File: kicad/capteur graphite CouBeh/capteur graphite CouBeh.kicad_pcb (KiCad board)
At the start: 2 copper layers, 68.6 x 53.3 mm, 23 parts, among them J1 Power, J2 Digital/PWM, J3 Analog, J4 Digital/PWM, J5 Conn_01x02, U2 LTC1050, U3 MCP41050

Commit message: Add files via upload
Routing:
- net +5V: track 123.4 -> 122.8 mm
- net BT RX: track 8.75 -> 9.35 mm

Commit message: Add files via upload
Parts:
- removed R1: 1k, Resistor_THT:R_Axial_DIN0204_L3.6mm_D1.6mm_P7.62mm_Horizontal
- moved U1 25.0 mm to (145.2, 88.0), turned to 180 degrees
- moved U3 1.69 mm to (125.5, 54.7)
Connections:
- C2 pad 1: Net-(U2--) -> Potar out
- R4 pad 1: Net-(U2--) -> Potar out
- U2 pad 2: Net-(U2--) -> Potar out
- U3 pad 1: PD SDI -> PD CS
- U3 pad 3: PD CS -> PD SDI
- U3 pad 4: unconnected-(U3-VSS-Pad4) -> GND
- U3 pad 5: unconnected-(U3-PA0-Pad5) -> GND
- U3 pad 6: unconnected-(U3-PW0-Pad6) -> GND
- U3 pad 7: unconnected-(U3-PB0-Pad7) -> Potar out
- U3 pad 8: unconnected-(U3-VDD-Pad8) -> +5V
Routing:
- net GND: track 48.7 -> 0.58 mm, vias 2 -> 0
- net Potar out: track 0.00 -> 35.3 mm
- net OLED SDA: track 51.7 -> 23.6 mm
- net PD SDI: track 12.7 -> 36.7 mm
- net OLED SCL: track 48.2 -> 24.3 mm
- net Net-(U2--): track 17.0 -> 0.00 mm
- net +5V: track 122.8 -> 138.9 mm
- net PD CS: track 22.7 -> 14.1 mm
- net PD SCK: track 11.3 -> 9.85 mm
